Commit message: feat: add RPLidar A2 sensor, brick walls world, updated RViz config

File: urdf/donar_robot.xacro (robot description, xacro)
@@ -2,5 +2,4 @@
 <robot name="donar_robot" xmlns:xacro="http://www.ros.org/wiki/xacro">
 <xacro:include filename="$(find donar_description)/urdf/materials.xacro" />
-<!-- BASE FOOTPRINT -->
 <!-- BASE FOOTPRINT -->
 <link name="base_footprint"/>
@@ -31,4 +30,32 @@
   </collision>
 </link>
+<!-- LIDAR SENSOR -->
+<xacro:property name="width" value="0.03815" />
+<xacro:property name="bodylen" value="0.041" />
+<link name="lidar_scanner">
+  <inertial>
+    <origin xyz="0.0 0.0 0.0" rpy="0 0 0"/>
+    <mass value="0.17"/>
+    <inertia ixx="0.0001" iyy="0.0001" izz="0.0001" ixy="0.0" iyz="0.0" ixz="0.0"/>
+  </inertial>
+  <visual>
+    <origin xyz="0.0 0.0 0.0" rpy="0 0 0"/>
+    <geometry>
+      <cylinder radius="${width}" length="${bodylen}"/>
+    </geometry>
+    <material name="black"/>
+  </visual>
+  <collision>
+    <origin xyz="0.0 0.0 0.0" rpy="0 0 0"/>
+    <geometry>
+      <cylinder radius="${width}" length="${bodylen}"/>
+    </geometry>
+  </collision>
+</link>
+<joint name="lidar_joint" type="fixed">
+  <origin xyz="0.00 0.00 0.41" rpy="0 0 0"/>
+  <parent link="base_link"/>
+  <child link="lidar_scanner"/>
+</joint>
 <!-- RIGHT WHEEL -->
 <link name="right_wheel_1">
@@ -184,4 +211,34 @@
   </plugin>
 </gazebo>
+<!-- RPLidar A2 -->
+<gazebo reference="lidar_scanner">
+  <material>Gazebo/Black</material>
+  <sensor type="gpu_lidar" name="RPLidar_A2_sensor">
+  <ignition_frame_id>lidar_scanner</ignition_frame_id>
+    <topic>/donar_robot/laser/scan</topic>
+    <visualize>true</visualize>
+    <update_rate>40</update_rate>
+    <ray>
+      <scan>
+        <horizontal>
+          <samples>720</samples>
+          <resolution>1</resolution>
+          <min_angle>-3.14159</min_angle>
+          <max_angle>3.14159</max_angle>
+        </horizontal>
+      </scan>
+      <range>
+        <min>0.20</min>
+        <max>16.0</max>
+        <resolution>0.02</resolution>
+      </range>
+      <noise>
+        <type>gaussian</type>
+        <mean>0.0</mean>
+        <stddev>0.01</stddev>
+      </noise>
+    </ray>
+  </sensor>
+</gazebo>
 <!-- GAZEBO MATERIALS -->
 <gazebo reference="base_link">

Commit message: feat: add RealSense D435, complete sensor suite, verified TF tree

File: urdf/donar_robot.xacro (robot description, xacro)
@@ -53,4 +53,105 @@
   </collision>
 </link>
+<!-- IntelRealSense D435 camera -->
+<!-- RGBD CAMERA -->
+<link name="camera_link">
+  <inertial>
+    <origin xyz="0 0 0" rpy="0 0 0"/>
+    <mass value="0.072"/>
+    <inertia ixx="0.000001" iyy="0.000001" izz="0.000001"
+             ixy="0.0" iyz="0.0" ixz="0.0"/>
+  </inertial>
+  <visual>
+    <origin xyz="0 0 0" rpy="0 0 0"/>
+  <geometry>
+    <box size="0.025 0.09 0.025"/>
+  </geometry>
+    <material name="black">
+      <color rgba="0.0 0.0 0.0 1.0"/>
+    </material>
+  </visual>
+  <collision>
+    <origin xyz="0 0 0" rpy="0 0 0"/>
+    <geometry>
+      <box size="0.09 0.025 0.025"/>
+    </geometry>
+  </collision>
+</link>
+<!-- Mount camera to robot -->
+<joint name="camera_joint" type="fixed">
+  <origin xyz="0.348 0.0 0.25" rpy="0 0 0"/>
+  <parent link="base_link"/>
+  <child link="camera_link"/>
+</joint>
+<!-- Optical frame - corrects coordinate convention -->
+<!-- ROS: X forward Y left Z up -->
+<!-- Camera optical: Z forward X right Y down -->
+<link name="camera_optical_frame"/>
+<joint name="camera_optical_joint" type="fixed">
+  <origin xyz="0 0 0" rpy="-1.5708 0 -1.5708"/>
+  <parent link="camera_link"/>
+  <child link="camera_optical_frame"/>
+</joint>
+<!-- GAZEBO SENSOR PLUGIN -->
+<gazebo reference="camera_link">
+  <sensor name="realsense_d435" type="rgbd_camera">
+    <!-- <ignition_frame_id>camera_optical_frame</ignition_frame_id> -->
+    <ignition_frame_id>camera_link</ignition_frame_id>
+    <camera name="realsense_d435">
+      <!-- D435 horizontal FOV: 91.2 degrees = 1.5908 radians -->
+      <horizontal_fov>1.5908</horizontal_fov>
+      <!-- Intrinsics calibrated for 1280x720 -->
+      <lens>
+        <intrinsics>
+          <fx>920.0</fx>
+          <fy>920.0</fy>
+          <cx>640.5</cx>
+          <cy>360.5</cy>
+          <s>0</s>
+        </intrinsics>
+      </lens>
+      <distortion>
+        <k1>0.096559</k1>
+        <k2>-0.237840</k2>
+        <k3>0.113659</k3>
+        <p1>0.000396</p1>
+        <p2>0.000247</p2>
+        <center>0.5 0.5</center>
+      </distortion>
+      <!-- Slight noise to simulate real sensor -->
+      <noise>
+        <type>gaussian</type>
+        <mean>0.0</mean>
+        <stddev>0.003</stddev>
+      </noise>
+      <!-- RGB image settings -->
+      <image>
+        <width>1280</width>
+        <height>720</height>
+        <format>RGB_INT8</format>
+      </image>
+      <!-- RGB clip -->
+      <clip>
+        <near>0.01</near>
+        <far>100</far>
+      </clip>
+      <!-- Depth clip — D435 spec: 0.1m to 10m -->
+      <depth_camera>
+        <clip>
+          <near>0.1</near>
+          <far>10.0</far>
+        </clip>
+      </depth_camera>
+    </camera>
+    <always_on>1</always_on>
+    <update_rate>30</update_rate>
+    <visualize>0</visualize>
+    <topic>/donar_robot/depth_camera</topic>
+  </sensor>
+</gazebo>
+<!-- Camera Gazebo material -->
+<gazebo reference="camera_link">
+  <material>Gazebo/White</material>
+</gazebo>
 <joint name="lidar_joint" type="fixed">
   <origin xyz="0.00 0.00 0.41" rpy="0 0 0"/>

Commit message: feat: add MPU9250 IMU sensor with Gazebo physics plugin

File: urdf/donar_robot.xacro (robot description, xacro)
@@ -53,4 +53,85 @@
   </collision>
 </link>
+<!--MPU9250 -->
+<link name="IMU_link">
+  <inertial>
+    <origin xyz="0 0 0" rpy="0 0 0"/>
+    <mass value="0.0005"/>
+    <inertia ixx="0.0000001" iyy="0.0000001" izz="0.0000001"
+             ixy="0.0" iyz="0.0" ixz="0.0"/>
+  </inertial>
+  <visual>
+    <origin xyz="0 0 0" rpy="0 0 0"/>
+  <geometry>
+    <box size="0.0025 0.009 0.0025"/>
+  </geometry>
+    <material name="black">
+      <color rgba="0.0 0.0 0.0 1.0"/>
+    </material>
+  </visual>
+  <collision>
+    <origin xyz="0 0 0" rpy="0 0 0"/>
+    <geometry>
+      <box size="0.0025 0.009 0.0025"/>
+    </geometry>
+  </collision>
+</link>
+<!-- Mount IMU to robot -->
+<joint name="IMU_joint" type="fixed">
+  <origin xyz="0.0 0.0 0.15" rpy="0 0 0"/>
+  <parent link="base_link"/>
+  <child link="IMU_link"/>
+</joint>
+<!-- GAZEBO SENSOR PLUGIN -->
+<gazebo reference="IMU_link">
+  <sensor name="mpu9250" type="imu">
+    <ignition_frame_id>IMU_link</ignition_frame_id>
+    <always_on>1</always_on>
+    <update_rate>100</update_rate>
+    <topic>/donar_robot/imu</topic>
+    <imu>
+      <angular_velocity>
+        <x>
+          <noise type="gaussian">
+            <mean>0.0</mean>
+            <stddev>0.00017</stddev>
+          </noise>
+        </x>
+        <y>
+          <noise type="gaussian">
+            <mean>0.0</mean>
+            <stddev>0.00017</stddev>
+          </noise>
+        </y>
+        <z>
+          <noise type="gaussian">
+            <mean>0.0</mean>
+            <stddev>0.00017</stddev>
+          </noise>
+        </z>
+      </angular_velocity>
+      <linear_acceleration>
+        <x>
+          <noise type="gaussian">
+            <mean>0.0</mean>
+            <stddev>0.0029</stddev>
+          </noise>
+        </x>
+        <y>
+          <noise type="gaussian">
+            <mean>0.0</mean>
+            <stddev>0.0029</stddev>
+          </noise>
+        </y>
+        <z>
+          <noise type="gaussian">
+            <mean>0.0</mean>
+            <stddev>0.0029</stddev>
+          </noise>
+        </z>
+      </linear_acceleration>
+    </imu>
+  </sensor>
+</gazebo>
 <!-- IntelRealSense D435 camera -->
 <!-- RGBD CAMERA -->
@@ -284,13 +365,4 @@
 </gazebo>
 <gazebo>
-  <plugin filename="ignition-gazebo-odometry-publisher-system"
-          name="ignition::gazebo::systems::OdometryPublisher">
-    <odom_topic>/donar_robot/odometry</odom_topic>
-    <odom_frame>odom</odom_frame>
-    <robot_base_frame>base_link</robot_base_frame>
-    <odom_publish_frequency>50</odom_publish_frequency>
-  </plugin>
-</gazebo>
-<gazebo>
   <plugin filename="ignition-gazebo-diff-drive-system"
           name="ignition::gazebo::systems::DiffDrive">
@@ -305,5 +377,5 @@
     <max_linear_acceleration>2.0</max_linear_acceleration>
     <topic>/donar_robot/cmd_vel</topic>
-    <odom_topic>odometry</odom_topic>
+    <odom_topic>/donar_robot/odometry</odom_topic>
     <frame_id>odom</frame_id>
     <child_frame_id>base_footprint</child_frame_id>
